File: hardware/led_ir_driver/led_ir_driver.kicad_sch (KiCad schematic)
At the start: 25 parts, among them J1 MCP4725 IR 0x60, J2 PI I2C INPUT / IR OUT, J3 MCP4725 RED 0x61, J5 IR LED A / K, J6 RED LED A / K, J7 5V INPUT / GND, Q1 2N4401 / E-B-C, Q2 2N4401 / E-B-C, U1 LM358P / DIP8 socket

Commit message: hardware: finalize LED IR driver v1.6 and audit MCP4725 wiring
Parts:
- added J4: RED DAC OUT / GND, TX:Header2, symbol TX:Conn2
- J2: footprint TX:Header6 -> TX:HeaderMixed
Connections:
- net DAC_RED: now also J4.1
- net GND: now also J4.2
Other:
- note added: "ADDR is configured on each module, not by this carrier PCB."
- note added: "Both GND pins share 0 V. OUT is a separate signal."
- note added: "For RED: remove the old ADDR-GND bridge before selecting VCC."
- note added: "J2: OUT/GND = 2.54 mm; SCL/SDA/3V3/GND = 2.00 mm"
- note added: "Matching labels connect SCL, SDA, 3V3 and GND between modules."
- note added: "Module ADDR: GND -> 0x60"
- note added: "Module ADDR: VCC -> 0x61"
- note removed: "C2/C4 optional. Removed: R5/R10, C1/C3, C6."
- note removed: "Crossings without dots = no connection."
- note removed: "Four shared nets above are NOT shorted to one another."

Commit message: hardware: use 100 ohm IR LED sense resistor
Parts:
- R4: value 82R 1% 0.25W -> 100R 1% 0.25W
Other:
- note removed: "I_LED approximately V_DAC / (2 x 82 ohm)"
Changed lines of the file:
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@@
 (symbol (lib_id "TX:R") (at 162.56 162.56 0) (unit 1) (in_bom yes) (on_board yes) (dnp no)
 (property "Reference" "R4" (at 170.18 160.02 0) (effects (font (size 1.1 1.1)) (justify left) ))
-(property "Value" "82R 1% 0.25W" (at 170.18 164.592 0) (effects (font (size 1.1 1.1)) (justify left) ))
+(property "Value" "100R 1% 0.25W" (at 170.18 164.592 0) (effects (font (size 1.1 1.1)) (justify left) ))
 (property "Footprint" "TX:R" (at 162.56 162.56 0) (effects (font (size 1.1 1.1)) (justify left) (hide yes)))
 (instances (project "led_ir_driver" (path "/6a15abe7-9d7a-52ab-a372-f3c70c0f892e" (reference "R4") (unit 1)))))
 (label "SENSE_IR" (at 119.38 147.32 0) (effects (font (size 1 1)) (justify left bottom)))
 (label "GND" (at 101.6 177.8 0) (effects (font (size 1 1)) (justify left bottom)))
-(text "I_LED approximately V_DAC / (2 x 82 ohm)" (at 109.22 187.96 0) (effects (font (size 1.27 1.27))))
+(text "I_LED approximately V_DAC / (2 x 100 ohm)" (at 109.22 187.96 0) (effects (font (size 1.27 1.27))))
 (symbol (lib_id "TX:C") (at 101.6 205.74 90) (unit 1) (in_bom yes) (on_board yes) (dnp yes)
 (property "Reference" "C2" (at 101.6 195.58 90) (effects (font (size 1.1 1.1))  ))
