File: hardware/led_ir_driver/led_ir_driver.kicad_sch (KiCad schematic)
At the start: 26 parts, among them J1 MCP4725 IR 0x60, J2 PI I2C INPUT / IR OUT, J3 MCP4725 RED 0x61, J4 RED DAC OUT / GND, J5 IR LED A / K, J6 RED LED A / K, J7 5V INPUT / GND, Q1 2N4401 / E-B-C, Q2 2N4401 / E-B-C, U1 LM358P / DIP8 socket

Commit message: Compact PPG boards, add receiver filters and package V-cut panel
Other:
- moved on the sheet: C5, C7, J6, J7, U1C

Commit message: Convert PPG passives to SMD and refresh compact V-cut panel
Parts:
- R4, R9: footprint TX:R -> TX:RSense
Changed lines of the file:
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@@
 (kicad_sch (version 20250114) (generator "eeschema") (paper "A3")
-(title_block (title "DATN: PPG-Simulator - LED / IR driver") (rev "1.7") (comment 1 "Nguyen Nhat Huy - Pham Thanh Vy"))
+(title_block (title "DATN: PPG-Simulator - LED / IR driver") (rev "1.8") (comment 1 "Nguyen Nhat Huy - Pham Thanh Vy"))
 (text "IR: MCP4725 0x60 -> LM358 -> 2N4401 -> LED" (at 101.6 15.24 0) (effects (font (size 1.4 1.4))))
 (symbol (lib_id "TX:Socket6") (at 38.1 50.8 0) (unit 1) (in_bom yes) (on_board yes) (dnp no)
@@
 (property "Reference" "R4" (at 170.18 160.02 0) (effects (font (size 1.1 1.1)) (justify left) ))
 (property "Value" "100R 1% 0.25W" (at 170.18 164.592 0) (effects (font (size 1.1 1.1)) (justify left) ))
-(property "Footprint" "TX:R" (at 162.56 162.56 0) (effects (font (size 1.1 1.1)) (justify left) (hide yes)))
+(property "Footprint" "TX:RSense" (at 162.56 162.56 0) (effects (font (size 1.1 1.1)) (justify left) (hide yes)))
 (instances (project "led_ir_driver" (path "/6a15abe7-9d7a-52ab-a372-f3c70c0f892e" (reference "R4") (unit 1)))))
 (label "SENSE_IR" (at 119.38 147.32 0) (effects (font (size 1 1)) (justify left bottom)))
@@
 (property "Reference" "R9" (at 373.38 160.02 0) (effects (font (size 1.1 1.1)) (justify left) ))
 (property "Value" "100R 1% 0.25W" (at 373.38 164.592 0) (effects (font (size 1.1 1.1)) (justify left) ))
-(property "Footprint" "TX:R" (at 365.76 162.56 0) (effects (font (size 1.1 1.1)) (justify left) (hide yes)))
+(property "Footprint" "TX:RSense" (at 365.76 162.56 0) (effects (font (size 1.1 1.1)) (justify left) (hide yes)))
 (instances (project "led_ir_driver" (path "/6a15abe7-9d7a-52ab-a372-f3c70c0f892e" (reference "R9") (unit 1)))))
 (label "SENSE_RED" (at 322.58 147.32 0) (effects (font (size 1 1)) (justify left bottom)))
