File: hardware/opt101_receiver_kicad/opt101_receiver/opt101_receiver.kicad_sch (KiCad schematic)
At the start: 11 parts, among them J1 A2 / RED, J2 A0 / IR, J3 ADS1115 outputs, U1 OPT101P, U2 OPT101P

Commit message: Compact PPG boards, add receiver filters and package V-cut panel
Parts:
- added C3, C4: 1uF X7R 16V, PPG:C0805_Hand, symbol PPG:C
- added R1, R2: 1k 1%, PPG:R0805_Hand, symbol PPG:R
Connections:
- net GND_IR: now also C4.2
- net GND_RED: now also C3.2
- net OUT_IR: now also C4.1, R2.2; no longer U2.4 (1M_FB), U2.5 (OUT)
- net OUT_RED: now also C3.1, R1.2; no longer U1.4 (1M_FB), U1.5 (OUT)
- new net RAW_IR: R2.1, U2.4 (1M_FB), U2.5 (OUT)
- new net RAW_RED: R1.1, U1.4 (1M_FB), U1.5 (OUT)
Other:
- note added: "R1/R2 + C3/C4: 1k / 1uF output low-pass, nominal fc = 159 Hz."
Changed lines of the file:
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@@
 (kicad_sch (version 20250114) (generator "eeschema") (paper "A4")
-(title_block (title "PPG - Dual OPT101P receiver") (date "2026-09-24") (rev "1.2") (comment 1 "70 x 32 mm / DIP-8 sockets / Grove A0 IR, A2 RED"))
+(title_block (title "PPG - Dual OPT101P receiver") (date "2026-09-24") (rev "1.3") (comment 1 "70 x 30 mm / DIP-8 sockets / Grove A0 IR, A2 RED"))
 (symbol (lib_id "PPG:OPT101P") (at 101.6 66.04 0) (unit 1) (in_bom yes) (on_board yes) (dnp no)
 (property "Reference" "U1" (at 101.6 52.040000000000006 0) (effects (font (size 1.1 1.1))  ))
@@
 (wire (pts (xy 114.3 73.66000000000001) (xy 124.46 73.66000000000001)) (stroke (width 0) (type default)))
 (wire (pts (xy 124.46 73.66000000000001) (xy 124.46 68.58000000000001)) (stroke (width 0) (type default)))
-(wire (pts (xy 124.46 68.58000000000001) (xy 147.32 68.58000000000001)) (stroke (width 0) (type default)))
+(wire (pts (xy 124.46 68.58000000000001) (xy 129.54 68.58000000000001)) (stroke (width 0) (type default)))
+(symbol (lib_id "PPG:R") (at 134.62 68.58000000000001 0) (unit 1) (in_bom yes) (on_board yes) (dnp no)
+(property "Reference" "R1" (at 134.62 61.58000000000001 0) (effects (font (size 1.1 1.1))  ))
+(property "Value" "1k 1%" (at 134.62 63.58000000000001 0) (effects (font (size 1.1 1.1))  ))
+(property "Footprint" "PPG:R0805_Hand" (at 134.62 63.58000000000001 0) (effects (font (size 1.1 1.1))  (hide yes)))
+(pin "1")
+(pin "2")
+(instances (project "opt101_receiver" (path "/c3c775c3-686a-5258-bf54-9a2dfbec053d" (reference "R1") (unit 1)))))
+(wire (pts (xy 139.7 68.58000000000001) (xy 147.32 68.58000000000001)) (stroke (width 0) (type default)))
 (wire (pts (xy 147.32 68.58000000000001) (xy 147.32 58.42000000000001)) (stroke (width 0) (type default)))
 (wire (pts (xy 147.32 58.42000000000001) (xy 167.64 58.42000000000001)) (stroke (width 0) (type default)))
-(label "OUT_RED" (at 124.46 68.58000000000001 0) (effects (font (size 1 1)) (justify left bottom)))
-(wire (pts (xy 124.46 73.66000000000001) (xy 124.46 81.28)) (stroke (width 0) (type default)))
-(wire (pts (xy 124.46 81.28) (xy 200.66 81.28)) (stroke (width 0) (type default)))
-(wire (pts (xy 200.66 81.28) (xy 200.66 99.06)) (stroke (width 0) (type default)))
+(label "RAW_RED" (at 124.46 68.58000000000001 0) (effects (font (size 1 1)) (justify left bottom)))
+(label "OUT_RED" (at 147.32 58.42000000000001 0) (effects (font (size 1 1)) (justify left bottom)))
+(wire (pts (xy 147.32 68.58000000000001) (xy 147.32 76.2)) (stroke (width 0) (type default)))
+(wire (pts (xy 147.32 76.2) (xy 200.66 76.2)) (stroke (width 0) (type default)))
+(symbol (lib_id "PPG:C") (at 134.62 81.28 0) (unit 1) (in_bom yes) (on_board yes) (dnp no)
+(property "Reference" "C3" (at 139.70000000000002 80.01 0) (effects (font (size 1.1 1.1)) (justify left) ))
+(property "Value" "1uF X7R 16V" (at 139.70000000000002 82.55 0) (effects (font (size 1.1 1.1)) (justify left) ))
+(property "Footprint" "PPG:C0805_Hand" (at 134.62 76.28 0) (effects (font (size 1.1 1.1)) (justify left) (hide yes)))
+(pin "1")
+(pin "2")
+(instances (project "opt101_receiver" (path "/c3c775c3-686a-5258-bf54-9a2dfbec053d" (reference "C3") (unit 1)))))
+(wire (pts (xy 139.7 68.58000000000001) (xy 139.7 74.93)) (stroke (width 0) (type default)))
+(wire (pts (xy 139.7 74.93) (xy 134.62 74.93)) (stroke (width 0) (type default)))
+(wire (pts (xy 134.62 74.93) (xy 134.62 77.47)) (stroke (width 0) (type default)))
+(wire (pts (xy 134.62 85.09) (xy 134.62 88.9)) (stroke (width 0) (type default)))
+(wire (pts (xy 200.66 76.2) (xy 200.66 99.06)) (stroke (width 0) (type default)))
 (wire (pts (xy 200.66 99.06) (xy 218.44 99.06)) (stroke (width 0) (type default)))
 (junction (at 73.66 43.18000000000001) (diameter 0) (color 0 0 0 0))
@@
 (junction (at 81.28 73.66000000000001) (diameter 0) (color 0 0 0 0))
 (junction (at 124.46 68.58000000000001) (diameter 0) (color 0 0 0 0))
-(junction (at 124.46 73.66000000000001) (diameter 0) (color 0 0 0 0))
+(junction (at 139.7 68.58000000000001) (diameter 0) (color 0 0 0 0))
+(junction (at 147.32 68.58000000000001) (diameter 0) (color 0 0 0 0))
+(junction (at 134.62 88.9) (diameter 0) (color 0 0 0 0))
 (text "RED: U1.4 -- U1.5 = internal 1 Mohm feedback" (at 119.38 96.52000000000001 0) (effects (font (size 1.1 1.1))))
 (symbol (lib_id "PPG:OPT101P") (at 101.6 132.08 0) (unit 1) (in_bom yes) (on_board yes) (dnp no)
@@
 (wire (pts (xy 114.3 139.70000000000002) (xy 124.46 139.70000000000002)) (stroke (width 0) (type default)))
 (wire (pts (xy 124.46 139.70000000000002) (xy 124.46 134.62)) (stroke (width 0) (type default)))
-(wire (pts (xy 124.46 134.62) (xy 147.32 134.62)) (stroke (width 0) (type default)))
+(wire (pts (xy 124.46 134.62) (xy 129.54 134.62)) (stroke (width 0) (type default)))
+(symbol (lib_id "PPG:R") (at 134.62 134.62 0) (unit 1) (in_bom yes) (on_board yes) (dnp no)
+(property "Reference" "R2" (at 134.62 127.62 0) (effects (font (size 1.1 1.1))  ))
+(property "Value" "1k 1%" (at 134.62 129.62 0) (effects (font (size 1.1 1.1))  ))
+(property "Footprint" "PPG:R0805_Hand" (at 134.62 129.62 0) (effects (font (size 1.1 1.1))  (hide yes)))
+(pin "1")
+(pin "2")
+(instances (project "opt101_receiver" (path "/c3c775c3-686a-5258-bf54-9a2dfbec053d" (reference "R2") (unit 1)))))
+(wire (pts (xy 139.7 134.62) (xy 147.32 134.62)) (stroke (width 0) (type default)))
 (wire (pts (xy 147.32 134.62) (xy 147.32 124.46000000000001)) (stroke (width 0) (type default)))
 (wire (pts (xy 147.32 124.46000000000001) (xy 167.64 124.46000000000001)) (stroke (width 0) (type default)))
-(label "OUT_IR" (at 124.46 134.62 0) (effects (font (size 1 1)) (justify left bottom)))
-(wire (pts (xy 124.46 139.70000000000002) (xy 124.46 147.32000000000002)) (stroke (width 0) (type default)))
-(wire (pts (xy 124.46 147.32000000000002) (xy 208.28 147.32000000000002)) (stroke (width 0) (type default)))
-(wire (pts (xy 208.28 147.32000000000002) (xy 208.28 104.14)) (stroke (width 0) (type default)))
+(label "RAW_IR" (at 124.46 134.62 0) (effects (font (size 1 1)) (justify left bottom)))
+(label "OUT_IR" (at 147.32 124.46000000000001 0) (effects (font (size 1 1)) (justify left bottom)))
+(wire (pts (xy 147.32 134.62) (xy 147.32 142.24)) (stroke (width 0) (type default)))
+(wire (pts (xy 147.32 142.24) (xy 208.28 142.24)) (stroke (width 0) (type default)))
+(symbol (lib_id "PPG:C") (at 134.62 147.32000000000002 0) (unit 1) (in_bom yes) (on_board yes) (dnp no)
+(property "Reference" "C4" (at 139.70000000000002 146.05 0) (effects (font (size 1.1 1.1)) (justify left) ))
+(property "Value" "1uF X7R 16V" (at 139.70000000000002 148.59000000000003 0) (effects (font (size 1.1 1.1)) (justify left) ))
+(property "Footprint" "PPG:C0805_Hand" (at 134.62 142.32000000000002 0) (effects (font (size 1.1 1.1)) (justify left) (hide yes)))
+(pin "1")
+(pin "2")
+(instances (project "opt101_receiver" (path "/c3c775c3-686a-5258-bf54-9a2dfbec053d" (reference "C4") (unit 1)))))
+(wire (pts (xy 139.7 134.62) (xy 139.7 140.97000000000003)) (stroke (width 0) (type default)))
+(wire (pts (xy 139.7 140.97000000000003) (xy 134.62 140.97000000000003)) (stroke (width 0) (type default)))
+(wire (pts (xy 134.62 140.97000000000003) (xy 134.62 143.51000000000002)) (stroke (width 0) (type default)))
+(wire (pts (xy 134.62 151.13000000000002) (xy 134.62 154.94)) (stroke (width 0) (type default)))
+(wire (pts (xy 208.28 142.24) (xy 208.28 104.14)) (stroke (width 0) (type default)))
 (wire (pts (xy 208.28 104.14) (xy 218.44 104.14)) (stroke (width 0) (type default)))
 (junction (at 73.66 109.22000000000001) (diameter 0) (color 0 0 0 0))
@@
 (junction (at 81.28 139.70000000000002) (diameter 0) (color 0 0 0 0))
 (junction (at 124.46 134.62) (diameter 0) (color 0 0 0 0))
-(junction (at 124.46 139.70000000000002) (diameter 0) (color 0 0 0 0))
+(junction (at 139.7 134.62) (diameter 0) (color 0 0 0 0))
+(junction (at 147.32 134.62) (diameter 0) (color 0 0 0 0))
+(junction (at 134.62 154.94) (diameter 0) (color 0 0 0 0))
 (text "IR: U2.4 -- U2.5 = internal 1 Mohm feedback" (at 119.38 162.56 0) (effects (font (size 1.1 1.1))))
 (symbol (lib_id "PPG:ADS_Output") (at 228.6 101.6 0) (unit 1) (in_bom yes) (on_board yes) (dnp no)
@@
 (text "Separate supply/return cables meet at the HAT. J3 has signals only: ADS must share HAT GND." (at 139.7 29.21 0) (effects (font (size 1.1 1.1))))
 (text "Crossings without dots are NOT connected. Pins 2, 6, 7 of OPT101 remain open." (at 139.7 35.56 0) (effects (font (size 1.1 1.1))))
+(text "R1/R2 + C3/C4: 1k / 1uF output low-pass, nominal fc = 159 Hz." (at 139.7 165.1 0) (effects (font (size 1.1 1.1))))
 (sheet_instances (path "/" (page "1")))
 )

Commit message: Convert PPG passives to SMD and refresh compact V-cut panel
Parts:
- C1, C2: footprint PPG:Bypass_100n_P2.5mm -> PPG:C0805_Hand
Changed lines of the file:
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@@
 (kicad_sch (version 20250114) (generator "eeschema") (paper "A4")
-(title_block (title "PPG - Dual OPT101P receiver") (date "2026-09-24") (rev "1.3") (comment 1 "70 x 30 mm / DIP-8 sockets / Grove A0 IR, A2 RED"))
+(title_block (title "PPG - Dual OPT101P receiver") (date "2026-09-24") (rev "1.4") (comment 1 "70 x 30 mm / DIP-8 sockets / Grove A0 IR, A2 RED"))
 (symbol (lib_id "PPG:OPT101P") (at 101.6 66.04 0) (unit 1) (in_bom yes) (on_board yes) (dnp no)
 (property "Reference" "U1" (at 101.6 52.040000000000006 0) (effects (font (size 1.1 1.1))  ))
@@
 (property "Reference" "C1" (at 53.339999999999996 64.77000000000001 0) (effects (font (size 1.1 1.1)) (justify left) ))
 (property "Value" "100nF 50V X7R ceramic" (at 53.339999999999996 67.31 0) (effects (font (size 1.1 1.1)) (justify left) ))
-(property "Footprint" "PPG:Bypass_100n_P2.5mm" (at 48.26 61.040000000000006 0) (effects (font (size 1.1 1.1)) (justify left) (hide yes)))
+(property "Footprint" "PPG:C0805_Hand" (at 48.26 61.040000000000006 0) (effects (font (size 1.1 1.1)) (justify left) (hide yes)))
 (pin "1")
 (pin "2")
@@
 (property "Reference" "C2" (at 53.339999999999996 130.81 0) (effects (font (size 1.1 1.1)) (justify left) ))
 (property "Value" "100nF 50V X7R ceramic" (at 53.339999999999996 133.35000000000002 0) (effects (font (size 1.1 1.1)) (justify left) ))
-(property "Footprint" "PPG:Bypass_100n_P2.5mm" (at 48.26 127.08000000000001 0) (effects (font (size 1.1 1.1)) (justify left) (hide yes)))
+(property "Footprint" "PPG:C0805_Hand" (at 48.26 127.08000000000001 0) (effects (font (size 1.1 1.1)) (justify left) (hide yes)))
 (pin "1")
 (pin "2")

Commit message: Shrink PPG receivers to 70x20 and driver to 70x40; refresh V-cut release
Parts:
- removed H1, H2, H3, H4: M3 / 3.2mm NPTH, PPG:MountingHole_M3, symbol PPG:MountingHole
Changed lines of the file:
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@@
 (kicad_sch (version 20250114) (generator "eeschema") (paper "A4")
-(title_block (title "PPG - Dual OPT101P receiver") (date "2026-09-24") (rev "1.4") (comment 1 "70 x 30 mm / DIP-8 sockets / Grove A0 IR, A2 RED"))
+(title_block (title "PPG - Dual OPT101P receiver") (date "2026-10-02") (rev "1.5") (comment 1 "70 x 20 mm / DIP-8 sockets / Grove A0 IR, A2 RED"))
 (symbol (lib_id "PPG:OPT101P") (at 101.6 66.04 0) (unit 1) (in_bom yes) (on_board yes) (dnp no)
 (property "Reference" "U1" (at 101.6 52.040000000000006 0) (effects (font (size 1.1 1.1))  ))
@@
 (pin "2")
 (instances (project "opt101_receiver" (path "/c3c775c3-686a-5258-bf54-9a2dfbec053d" (reference "J3") (unit 1)))))
-(symbol (lib_id "PPG:MountingHole") (at 30.48 180.34 0) (unit 1) (in_bom yes) (on_board yes) (dnp no)
-(property "Reference" "H1" (at 30.48 173.34 0) (effects (font (size 1.1 1.1))  ))
-(property "Value" "M3 / 3.2mm NPTH" (at 30.48 175.34 0) (effects (font (size 1.1 1.1))  ))
-(property "Footprint" "PPG:MountingHole_M3" (at 30.48 175.34 0) (effects (font (size 1.1 1.1))  (hide yes)))
-(instances (project "opt101_receiver" (path "/c3c775c3-686a-5258-bf54-9a2dfbec053d" (reference "H1") (unit 1)))))
-(symbol (lib_id "PPG:MountingHole") (at 71.12 180.34 0) (unit 1) (in_bom yes) (on_board yes) (dnp no)
-(property "Reference" "H2" (at 71.12 173.34 0) (effects (font (size 1.1 1.1))  ))
-(property "Value" "M3 / 3.2mm NPTH" (at 71.12 175.34 0) (effects (font (size 1.1 1.1))  ))
-(property "Footprint" "PPG:MountingHole_M3" (at 71.12 175.34 0) (effects (font (size 1.1 1.1))  (hide yes)))
-(instances (project "opt101_receiver" (path "/c3c775c3-686a-5258-bf54-9a2dfbec053d" (reference "H2") (unit 1)))))
-(symbol (lib_id "PPG:MountingHole") (at 111.76 180.34 0) (unit 1) (in_bom yes) (on_board yes) (dnp no)
-(property "Reference" "H3" (at 111.76 173.34 0) (effects (font (size 1.1 1.1))  ))
-(property "Value" "M3 / 3.2mm NPTH" (at 111.76 175.34 0) (effects (font (size 1.1 1.1))  ))
-(property "Footprint" "PPG:MountingHole_M3" (at 111.76 175.34 0) (effects (font (size 1.1 1.1))  (hide yes)))
-(instances (project "opt101_receiver" (path "/c3c775c3-686a-5258-bf54-9a2dfbec053d" (reference "H3") (unit 1)))))
-(symbol (lib_id "PPG:MountingHole") (at 152.4 180.34 0) (unit 1) (in_bom yes) (on_board yes) (dnp no)
-(property "Reference" "H4" (at 152.4 173.34 0) (effects (font (size 1.1 1.1))  ))
-(property "Value" "M3 / 3.2mm NPTH" (at 152.4 175.34 0) (effects (font (size 1.1 1.1))  ))
-(property "Footprint" "PPG:MountingHole_M3" (at 152.4 175.34 0) (effects (font (size 1.1 1.1))  (hide yes)))
-(instances (project "opt101_receiver" (path "/c3c775c3-686a-5258-bf54-9a2dfbec053d" (reference "H4") (unit 1)))))
 (text "DUAL OPT101 RECEIVER: RED -> A2 / IR -> A0" (at 139.7 15.24 0) (effects (font (size 1.7 1.7))))
 (text "3.3 V only. C1/C2: non-polar ceramic 100 nF, X7R, 50 V." (at 139.7 22.86 0) (effects (font (size 1.2 1.2))))
